Commit message: add upper and lower joint angle limits

File: urdf/robot_arm_urdf.urdf (robot description, URDF)
Before this commit: robot robot_arm_urdf, 4 links, 3 joints
Joints:
- joint lowerLinkJoint: limit lower=0 upper=0 effort=1 velocity=1 -> lower=-3.14 upper=3.14 effort=1 velocity=1; type continuous -> revolute
- joint midLinkJoint: limit lower=0 upper=0 effort=1 velocity=1 -> lower=-3.14 upper=3.14 effort=10 velocity=1
- joint topLinkJoint: limit lower=0 upper=0 effort=1 velocity=1 -> lower=-3.14 upper=3.14 effort=1 velocity=1
